File: MicrocontrollerBoard/puenteH/puenteH.sch (KiCad schematic (older format))
At the start: 47 parts, among them J1 PROG_CONN, J10 PCA_5V, J11 PCB_5V, J12 PDA_5V, J13 PA_GND, J14 PBA_GND, J15 PCA_GND, J16 PCB_GND, J17 PDA_GND, J18 COM, J19 COM_5V, J2 5V_CONN, J20 COM_GND, J21 POWER_CONN, J22 MOTOR2, J23 MOTOR1, J3 PA, J4 PBA, J5 PCA, J6 PCB, J7 PDA, J8 PA_5V, J9 PBA_5V, U1 ATmega1284P-PU, U2 TC4422, U3 TC4422, U4 TC4422, U5 TC4422, Y1 16MHz

Commit message: Microcontroller bord: Fixed PWM lines not going to uc's PWM pins. Added 3V3 regulator.
Parts:
- removed J11: PCB_5V, Connector_PinHeader_2.54mm:PinHeader_1x02_P2.54mm_Vertical, symbol Connector_Generic:Conn_01x02
- removed J12: PDA_5V, Connector_PinHeader_2.54mm:PinHeader_1x04_P2.54mm_Vertical, symbol Connector_Generic:Conn_01x04
- removed J16: PCB_GND, Connector_PinHeader_2.54mm:PinHeader_1x02_P2.54mm_Vertical, symbol Connector_Generic:Conn_01x02
- removed J17: PDA_GND, Connector_PinHeader_2.54mm:PinHeader_1x04_P2.54mm_Vertical, symbol Connector_Generic:Conn_01x04
- removed J7: PDA, Connector_PinHeader_2.54mm:PinHeader_1x04_P2.54mm_Vertical, symbol Connector_Generic:Conn_01x04
- added C4, C7: 100uF, Capacitor_THT:CP_Radial_D5.0mm_P2.50mm, symbol Device:CP
- added C5, C6: 100nF, Capacitor_SMD:C_0603_1608Metric_Pad1.05x0.95mm_HandSolder, symbol Device:C
- added J7: 3V_CONN_2, Connector_PinHeader_2.54mm:PinHeader_1x02_P2.54mm_Vertical, symbol Connector_Generic:Conn_01x02
- added U6: AMS1117-3.3, Package_TO_SOT_SMD:SOT-223-3_TabPin2, symbol Regulator_Linear:AMS1117-3.3
- J10: value PCA_5V -> PC_5V; footprint Connector_PinHeader_2.54mm:PinHeader_1x02_P2.54mm_Vertical -> Connector_PinHeader_2.54mm:PinHeader_1x08_P2.54mm_Vertical; symbol Connector_Generic:Conn_01x02 -> Connector_Generic:Conn_01x08
- J14: value PBA_GND -> PB_GND
- J15: value PCA_GND -> PC_GND; footprint Connector_PinHeader_2.54mm:PinHeader_1x02_P2.54mm_Vertical -> Connector_PinHeader_2.54mm:PinHeader_1x08_P2.54mm_Vertical; symbol Connector_Generic:Conn_01x02 -> Connector_Generic:Conn_01x08
- J4: value PBA -> PB
- J5: value PCA -> PC; footprint Connector_PinHeader_2.54mm:PinHeader_1x02_P2.54mm_Vertical -> Connector_PinHeader_2.54mm:PinHeader_1x08_P2.54mm_Vertical; symbol Connector_Generic:Conn_01x02 -> Connector_Generic:Conn_01x08
- J6: value PCB -> 3V_CONN_1
- J9: value PBA_5V -> PB_5V
Connections:
- net +5V: now also J10.3 (Pin_3), J10.4 (Pin_4), J10.5 (Pin_5), J10.6 (Pin_6), J10.7 (Pin_7), J10.8 (Pin_8), C4.1, C5.1, U6.3 (VI)
- net GND: now also J15.3 (Pin_3), J15.4 (Pin_4), J15.5 (Pin_5), J15.6 (Pin_6), J15.7 (Pin_7), J15.8 (Pin_8), J6.2 (Pin_2), C4.2, C5.2, C6.2, C7.2, J7.2 (Pin_2), U6.1 (GND)
- net MOTOR1A: now also U1.20 (PD6); no longer U1.24 (PC2)
- net MOTOR1B: now also U1.19 (PD5); no longer U1.25 (PC3)
- net MOTOR2A: now also U1.18 (PD4); no longer U1.26 (PC4)
- net MOTOR2B: now also U1.21 (PD7); no longer U1.27 (PC5)
- net at U1.28 (PC6): now also J5.7 (Pin_7); no longer J6.1 (Pin_1)
- net at U1.29 (PC7): now also J5.8 (Pin_8); no longer J6.2 (Pin_2)
- new net: J5.3 (Pin_3), U1.24 (PC2)
- new net: J5.4 (Pin_4), U1.25 (PC3)
- new net: J5.5 (Pin_5), U1.26 (PC4)
- new net: J5.6 (Pin_6), U1.27 (PC5)
- new net: C6.1, C7.1, J6.1 (Pin_1), J7.1 (Pin_1), U6.2 (VO)
